File: PCB_Shield/PCB_Shield.sch (KiCad schematic (older format))
At the start: 22 parts, among them P1 Power, P2 Analog, P3 Digital, P4 Digital, P5 CONN_01X01, P6 CONN_01X01, P7 CONN_01X01, P8 CONN_01X01, U0 CG, U1 LTC1050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

Commit message: Modif_10-03-2021
Connections:
- net SCL: now also P2.6 (Pin_6), P3.1 (Pin_1); no longer P2.5 (Pin_5), P3.2 (Pin_2)
- net SDA: now also P2.5 (Pin_5), P3.2 (Pin_2); no longer P2.6 (Pin_6), P3.1 (Pin_1)
Changed lines of the file:
@@
 Wire Wire Line
 	4750 5050 5500 5050
-Text GLabel 8750 2900 0    50   Input ~ 0
-SCL
-Text GLabel 8750 3000 0    50   Input ~ 0
-SDA
 Wire Wire Line
 	8750 2900 9400 2900
@@
 Wire Wire Line
 	10200 2500 10550 2500
+Text GLabel 8750 2900 0    50   Input ~ 0
+SDA
+Text GLabel 8750 3000 0    50   Input ~ 0
+SCL
 $EndSCHEMATC
