File: PCB_Shield/PCB_Shield.kicad_pcb (KiCad board)
At the start: 2 copper layers, 68.6 x 53.3 mm, 22 parts, among them P1 Power, P2 Analog, P3 Digital, P4 Digital, P5 CONN_01X01, P6 CONN_01X01, P7 CONN_01X01, P8 CONN_01X01, U0 CG, U1 LTC1050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

Commit message: Modification PCB _ test routage
Parts:
- moved C3 25.4 mm to (159.0, 94.1), turned to 180 degrees
- moved R2 23.8 mm to (142.5, 107.3), turned to 180 degrees
- moved C2 18.7 mm to (161.0, 117.5), turned to 0 degrees
- moved U1 11.2 mm to (120.9, 105.0), turned to 90 degrees
- moved R3 10.9 mm to (139.7, 90.3), turned to 180 degrees
- moved R6 9.55 mm to (160.8, 113.2)
- moved C4 8.39 mm to (137.2, 85.0), turned to 180 degrees
- moved C1 4.33 mm to (134.6, 114.9)
- moved U0 4.20 mm to (117.1, 98.4)
- moved R1 3.66 mm to (130.8, 114.7)
- moved R5 0.51 mm to (128.5, 111.6)
Routing:
- net +5V: track 0.00 -> 110.7 mm
- net Net-(C4-Pad1): track 0.00 -> 68.0 mm
- net Net-(C4-Pad2): track 0.00 -> 46.8 mm
- net Net-(C1-Pad1): track 0.00 -> 15.8 mm
- net Net-(R5-Pad2): track 0.00 -> 11.7 mm
- net ADC: track 0.00 -> 11.1 mm
- net Rx: track 1.52 -> 10.9 mm
- net Tx: track 2.35 -> 11.4 mm
- net GND: track 39.3 -> 43.8 mm
- net CLK: track 31.8 -> 33.1 mm

Commit message: Modif_PCB_Nom
Other:
- board text added: "GR1_Binome6"
Changed lines of the file:
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@@
   (general
     (thickness 1.6)
-    (drawings 27)
+    (drawings 28)
     (tracks 102)
     (zones 0)
@@
   (page A4)
   (title_block
-    (date "lun. 30 mars 2015")
+    (title Shield_Capteur_Graphite_Arduino_UNO)
+    (date 2021-03-09)
+    (company "INSA Toulouse")
+    (comment 1 Gaich&Stephen)
   )
   (layers
@@
       (effects (font (size 1 1) (thickness 0.15)))
     )
-    (fp_text user %R (at 5.08 0) (layer F.Fab)
-      (effects (font (size 1 1) (thickness 0.15)))
-    )
     (fp_line (start 11.21 -1.5) (end -1.05 -1.5) (layer F.CrtYd) (width 0.05))
     (fp_line (start 11.21 1.5) (end 11.21 -1.5) (layer F.CrtYd) (width 0.05))
@@
     (fp_line (start 1.93 1.25) (end 8.23 1.25) (layer F.Fab) (width 0.1))
     (fp_line (start 1.93 -1.25) (end 1.93 1.25) (layer F.Fab) (width 0.1))
+    (fp_text user %R (at 5.08 0) (layer F.Fab)
+      (effects (font (size 1 1) (thickness 0.15)))
+    )
     (pad 2 thru_hole oval (at 10.16 0 180) (size 1.6 1.6) (drill 0.8) (layers *.Cu *.Mask)
       (net 28 "Net-(C4-Pad2)"))
@@
       (net 4 GND))
   )
+  (gr_text GR1_Binome6 (at 171.704 86.995 90) (layer B.Cu)
+    (effects (font (size 1.5 1.5) (thickness 0.3)) (justify mirror))
+  )
   (gr_text 1 (at 138.938 121.285 90) (layer F.SilkS)

Commit message: Modification_TD
Parts:
- moved C4 11.0 mm to (128.5, 91.8)
- moved R3 6.36 mm to (133.3, 90.6), turned to 270 degrees
- moved U4 3.14 mm to (163.6, 104.3)
- moved U3 2.87 mm to (175.0, 107.8), turned to 90 degrees
Routing:
- net GND: track 43.8 -> 61.4 mm
- net SDA: track 12.5 -> 23.4 mm
- net Net-(C4-Pad1): track 68.0 -> 57.2 mm
- net Net-(C4-Pad2): track 46.8 -> 41.2 mm
- net SCL: track 15.5 -> 20.7 mm
- net SWITCH: track 32.8 -> 29.4 mm
- net DATA: track 32.8 -> 29.4 mm
- net CLK: track 33.1 -> 31.2 mm
- net +5V: track 110.7 -> 112.2 mm
Other:
- net class Default: clearance 0.8 -> 0.5
- rule trace_clearance: 0.8 -> 0.5

Commit message: Ajout
Connections:
- P4 pad 3: SWITCH -> /5(**)
- P4 pad 5: /3(**) -> CLK
- P4 pad 6: CLK -> SWITCH
Routing:
- net SWITCH: track 29.4 -> 38.9 mm
- net CLK: track 31.2 -> 29.4 mm
Other:
- net class Default: clearance 0.5 -> 0.4
- rule trace_clearance: 0.5 -> 0.4
- rule trace_min: 0.2 -> 0.8

Commit message: Modif_10-03-2021
Parts:
- moved U3 2.74 mm to (174.0, 110.4), turned to 270 degrees
- moved U4 1.27 mm to (162.3, 104.3)
- moved R1 0.57 mm to (131.3, 114.4)
- moved C1 0.51 mm to (135.1, 114.9)
Connections:
- P2 pad 5: SCL -> SDA
- P2 pad 6: SDA -> SCL
- P3 pad 1: SDA -> SCL
- P3 pad 2: SCL -> SDA
Routing:
- net SDA: track 23.4 -> 10.5 mm
- net SCL: track 20.7 -> 14.1 mm
- net GND: track 61.4 -> 56.3 mm
- net +5V: track 112.2 -> 108.6 mm
- net Net-(C1-Pad1): track 15.8 -> 18.2 mm
- net Tx: track 11.4 -> 13.0 mm
- net Net-(C4-Pad2): track 41.2 -> 42.3 mm
- net SWITCH: track 38.9 -> 39.9 mm
Other:
- outline, holes or cut-outs redrawn
